File: hardware/rgbcp.sch (KiCad schematic (older format))
At the start: 166 parts, among them SW0 SW_PUSH, SW1 SW_PUSH, SW2 SW_PUSH, SW3 SW_PUSH, SW4 SW_PUSH, SW5 SW_PUSH

Commit message: fix #2, #7: Use MAX603ESA Instead of 4-7V
Parts:
- removed BJTA1B, BJTA1G, BJTA1R, BJTA2B, BJTA2G, BJTA2R, BJTA3B, BJTA3G, BJTA3R, BJTBT0, BJTBT1, BJTBT2, BJTBT3, BJTDB, BJTDG, BJTDR: BCP56-16, symbol NPN
- removed R? (x10): 270, symbol R
- removed R? (x6): 220, symbol R
- added C? (x2): 10uF, symbol CP1
- added R?: 1.1M, symbol R
- added R?: 470K, symbol R
- added U?: MAX603ESA, symbol MAX603ESA
- R? (x9): value 270 -> 180
Connections:
- net A_LED1B: now also R?.1
- net A_LED1G: now also R?.1
- net A_LED1R: now also R?.1
- net A_LED2B: now also R?.1
- net A_LED2G: now also R?.1
- net A_LED2R: now also R?.1
- net A_LED3B: now also R?.1
- net A_LED3G: now also R?.1
- net A_LED3R: now also R?.1
- net GND: now also C?.2, C?.2, R?.2, U?.2 (GND), U?.3 (GND), U?.6 (GND), U?.7 (GND)
- net LED_BAT_0: now also R?.1
- net LED_BAT_1: now also R?.1
- net LED_BAT_2: now also R?.1
- net LED_BAT_3: now also R?.1
- net LED_DBG_B: now also R?.1
- net LED_DBG_G: now also R?.1
- net LED_DBG_R: now also R?.1
- net VIN_4-7V: now also C?.1, U?.1 (IN), U?.4 (~OFF); no longer BJTCS0.3 (C), BJTCS1.3 (C), BJTCS2.3 (C), BJTCS3.3 (C), BJTCS4.3 (C), BJTCS5.3 (C), BJTCS6.3 (C), BJTCS7.3 (C), BJTCS8.3 (C), BJTCS9.3 (C), LEDBAT0.1 (A), LEDBAT1.1 (A), LEDBAT2.1 (A), LEDBAT3.1 (A), LEDDBG.CA
- new net: R?.1, R?.2, U?.5 (SET)
- new net STAB_4V: BJTCS0.3 (C), BJTCS1.3 (C), BJTCS2.3 (C), BJTCS3.3 (C), BJTCS4.3 (C), BJTCS5.3 (C), BJTCS6.3 (C), BJTCS7.3 (C), BJTCS8.3 (C), BJTCS9.3 (C), C?.1, LEDBAT0.1 (A), LEDBAT1.1 (A), LEDBAT2.1 (A), LEDBAT3.1 (A), LEDDBG.CA, R?.1, U?.8 (OUT)
Other:
- moved on the sheet: R?
